File: Arduino.kicad_sch (KiCad schematic)
At the start: 27 parts, among them J1 Analog Pins, J2 Digital Pins, J3 Digital Pins, J4 ICSP, J5 Barrel_Jack_Switch, J6 Conector, J7 PWR, J8 USB_B, SW1 SW_SPST, U1 ATmega328P-P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

Commit message: Adding final version
Parts:
- C5: value 100 nF -> 0.1uF
- C6: value 47 uF -> 100uF/25V
Connections:
- net USB_5V: no longer U2.8 (VBUS)
- net VCC: now also J6.2 (Pin_2), U2.8 (VBUS)
- net VIN: no longer J6.2 (Pin_2)
Changed lines of the file:
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@@
 	(wire
 		(pts
-			(xy 101.6 44.45) (xy 85.09 44.45)
-		)
-		(stroke
-			(width 0)
-			(type default)
-		)
-	)
-	(wire
-		(pts
-			(xy 107.95 49.53) (xy 101.6 49.53)
-		)
-		(stroke
-			(width 0)
-			(type default)
-		)
-	)
-	(wire
-		(pts
 			(xy 219.71 88.9) (xy 215.9 88.9)
 		)
@@
 	(wire
 		(pts
-			(xy 101.6 49.53) (xy 101.6 44.45)
-		)
-		(stroke
-			(width 0)
-			(type default)
-		)
-	)
-	(wire
-		(pts
 			(xy 200.66 71.12) (xy 214.63 71.12)
 		)
@@
 	)
 	(label "USB_5V"
-		(at 93.98 44.45 0)
-		(fields_autoplaced yes)
-		(effects
-			(font
-				(size 1.27 1.27)
-			)
-			(justify left bottom)
-		)
-	)
-	(label "VIN"
-		(at 52.07 177.8 0)
+		(at 85.09 44.45 0)
 		(fields_autoplaced yes)
 		(effects
@@
 	)
 	(symbol
+		(lib_id "power:VCC")
+		(at 107.95 49.53 90)
+		(unit 1)
+		(exclude_from_sim no)
+		(in_bom yes)
+		(on_board yes)
+		(dnp no)
+		(fields_autoplaced yes)
+		(property "Reference" "#PWR021"
+			(at 111.76 49.53 0)
+			(effects
+				(font
+					(size 1.27 1.27)
+				)
+				(hide yes)
+			)
+		)
+		(property "Value" "VCC"
+			(at 104.14 49.5299 90)
+			(effects
+				(font
+					(size 1.27 1.27)
+				)
+				(justify left)
+			)
+		)
+		(property "Footprint" ""
+			(at 107.95 49.53 0)
+			(effects
+				(font
+					(size 1.27 1.27)
+				)
+				(hide yes)
+			)
+		)
+		(property "Datasheet" ""
+			(at 107.95 49.53 0)
+			(effects
+				(font
+					(size 1.27 1.27)
+				)
+				(hide yes)
+			)
+		)
+		(property "Description" "Power symbol creates a global label with name \"VCC\""
+			(at 107.95 49.53 0)
+			(effects
+				(font
+					(size 1.27 1.27)
+				)
+				(hide yes)
+			)
+		)
+		(pin "1"
+		)
+		(instances
+			(project ""
+				(path "/5adcfd62-53cf-4dcb-bfbf-d2207db0650f"
+					(reference "#PWR021")
+					(unit 1)
+				)
+			)
+		)
+	)
+	(symbol
 		(lib_id "Interface_USB:CP2102N-Axx-xQFN28")
 		(at 120.65 64.77 0)
@@
 	)
 	(symbol
+		(lib_id "power:VCC")
+		(at 52.07 177.8 270)
+		(unit 1)
+		(exclude_from_sim no)
+		(in_bom yes)
+		(on_board yes)
+		(dnp no)
+		(fields_autoplaced yes)
+		(property "Reference" "#PWR014"
+			(at 48.26 177.8 0)
+			(effects
+				(font
+					(size 1.27 1.27)
+				)
+				(hide yes)
+			)
+		)
+		(property "Value" "VCC"
+			(at 55.88 177.7999 90)
+			(effects
+				(font
+					(size 1.27 1.27)
+				)
+				(justify left)
+			)
+		)
+		(property "Footprint" ""
+			(at 52.07 177.8 0)
+			(effects
+				(font
+					(size 1.27 1.27)
+				)
+				(hide yes)
+			)
+		)
+		(property "Datasheet" ""
+			(at 52.07 177.8 0)
+			(effects
+				(font
+					(size 1.27 1.27)
+				)
+				(hide yes)
+			)
+		)
+		(property "Description" "Power symbol creates a global label with name \"VCC\""
+			(at 52.07 177.8 0)
+			(effects
+				(font
+					(size 1.27 1.27)
+				)
+				(hide yes)
+			)
+		)
+		(pin "1"
+		)
+		(instances
+			(project ""
+				(path "/5adcfd62-53cf-4dcb-bfbf-d2207db0650f"
+					(reference "#PWR014")
+					(unit 1)
+				)
+			)
+		)
+	)
+	(symbol
 		(lib_id "Device:Crystal")
 		(at 219.71 85.09 90)
@@
 			)
 		)
-		(property "Value" "47 uF"
+		(property "Value" "100uF/25V"
 			(at 83.82 157.8609 0)
 			(effects
@@
 			)
 		)
-		(property "Value" "100 nF"
+		(property "Value" "0.1uF"
 			(at 69.85 158.7499 0)
 			(effects
