File: Arduino.kicad_pcb (KiCad board)
At the start: 2 copper layers, 68 x 53 mm, 27 parts, among them J1 Analog Pins, J2 Digital Pins, J3 Digital Pins, J4 ICSP, J5 Barrel_Jack_Switch, J6 Conector, J7 PWR, J8 USB_B, SW1 SW_SPST, U1 ATmega328P-P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

Commit message: Fixed small mistake
Routing:
- net GND: track 259.0 -> 255.6 mm
Changed lines of the file:
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@@
 		)
 		(pad "2" thru_hole circle
-			(at 2.75 -2.25)
+			(at -2.75 2.25)
 			(size 1.524 1.524)
 			(drill 0.762)
@@
 		)
 		(pad "4" thru_hole circle
-			(at -2.7 2.25)
+			(at 2.75 -2.25)
 			(size 1.524 1.524)
 			(drill 0.762)
@@
 	)
 	(segment
-		(start 122.25 76.2)
-		(end 125.35 79.3)
-		(width 0.7)
-		(layer "F.Cu")
-		(net 2)
-	)
-	(segment
 		(start 127.94 108.31)
 		(end 116.25 108.31)
@@
 		(start 115.85 84.444551)
 		(end 116.994551 83.3)
-		(width 0.7)
-		(layer "F.Cu")
-		(net 2)
-	)
-	(segment
-		(start 125.35 79.3)
-		(end 125.35 83.3)
 		(width 0.7)
 		(layer "F.Cu")
@@
 		(layer "F.Cu")
 		(net 2)
+	)
+	(segment
+		(start 115.85 85.76)
+		(end 115.85 80.8)
+		(width 0.5)
+		(layer "F.Cu")
+		(net 2)
